File: Projects/555Timer/555Timer.kicad_pcb (KiCad board)
At the start: 2 copper layers, 39.9 x 30 mm, 14 parts, among them J1 Conn_01x04_Pin, U1 LM555xN

Commit message: Updte
Parts:
- removed the REF** at (79.9, 54.0)
- removed the REF** at (79.9, 78.0)
- removed the REF** at (113.9, 78.0)
- removed the REF** at (113.9, 54.0)
- added REF**: MountingHole_2.2mm_M2, MountingHole:MountingHole_2.2mm_M2, F.Cu at (113.0, 54.0)
- added REF**: MountingHole_2.2mm_M2, MountingHole:MountingHole_2.2mm_M2, F.Cu at (113.0, 78.0)
- added REF**: MountingHole_2.2mm_M2, MountingHole:MountingHole_2.2mm_M2, F.Cu at (79.0, 78.0)
- added REF**: MountingHole_2.2mm_M2, MountingHole:MountingHole_2.2mm_M2, F.Cu at (79.0, 54.0)
- moved C1 5.36 mm to (104.0, 55.0), turned to -90 degrees
- moved D1 4.44 mm to (95.0, 55.0), turned to -90 degrees
- moved C2 1.00 mm to (110.9, 63.0)
Routing:
- net Net-(U1-CV): track 20.5 -> 8.59 mm
- net GND: track 85.6 -> 92.5 mm
- net THR: track 28.7 -> 33.3 mm
- net VCC: track 39.0 -> 41.0 mm
- net Net-(D1-A): track 2.65 -> 3.86 mm
- net OUT1: track 25.3 -> 26.3 mm
- removed copper zone on B.Cu, net GND
Other:
- board text added: "555 Timer"
- board text added: "BS170"
- board text added: "C1 0.1µF"
- board text added: "C22 100µF"
- board text added: "GND"
- board text added: "LM555 DIP"
- board text added: "NNM22AM033"
- board text added: "OUT1"
- board text added: "OUT2"
- board text added: "PWR LED"
- board text added: "R1 220Ω"
- board text added: "R2 1kΩ"
- board text added: "R3 100kΩ"
- board text added: "R4 10kΩ"
