File: Projects/555Timer/555Timer.kicad_sch (KiCad schematic)
At the start: 10 parts, among them J1 Conn_01x04_Pin, U1 LM555xN

Commit message: Update
Parts:
- C1: footprint (none) -> Capacitor_THT:C_Disc_D5.0mm_W2.5mm_P5.00mm
- C2: footprint (none) -> Capacitor_THT:CP_Radial_Tantal_D5.0mm_P2.50mm
- D1: footprint (none) -> LED_THT:LED_D3.0mm
- J1: footprint (none) -> Connector_PinSocket_2.54mm:PinSocket_1x04_P2.54mm_Vertical
- R1, R2, R3, R4: footprint (none) -> Resistor_THT:R_Axial_DIN0204_L3.6mm_D1.6mm_P7.62mm_Horizontal
- renumbered MOSFET to MOSFET1
Other:
- company: (none) -> Nandan R Pai
- title: (none) -> 555 Timer Circuit
- moved on the sheet: C1, C2, D1, J1, MOSFET1, R1, R2, R3, R4, U1

Commit message: Updte
Parts:
- R1: value 220 -> 220Ω
Changed lines of the file:
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@@
 		(fields_autoplaced yes)
 		(property "Reference" "R1"
-			(at 52.07 48.26 90)
+			(at 48.26 46.9899 0)
 			(effects
 				(font
 					(size 1.27 1.27)
 				)
+				(justify right)
 			)
 		)
-		(property "Value" "220"
-			(at 49.53 48.26 90)
+		(property "Value" "220Ω"
+			(at 48.26 49.5299 0)
 			(effects
 				(font
 					(size 1.27 1.27)
 				)
+				(justify right)
 			)
 		)
