File: Projects/MotorController/_autosave-MotorController.kicad_sch (KiCad schematic)
At the start: 20 parts, among them J2 Conn_01x03_Pin, J3 Conn_01x03_Pin, J4 Screw_Terminal_01x02, J5 Screw_Terminal_01x02, SW1 SW_SPST, U1 L7805, U2 L298N

Commit message: Motor Controller
Parts:
- J4, J5: footprint TerminalBlock_Altech:Altech_AK100_1x02_P5.00mm -> TerminalBlock:TerminalBlock_Altech_AK300-2_P5.00mm
Changed lines of the file:
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@@
 			)
 		)
-		(property "Footprint" "TerminalBlock_Altech:Altech_AK100_1x02_P5.00mm"
+		(property "Footprint" "TerminalBlock:TerminalBlock_Altech_AK300-2_P5.00mm"
 			(at 205.74 116.84 0)
 			(effects
@@
 			)
 		)
-		(property "Footprint" "TerminalBlock_Altech:Altech_AK100_1x02_P5.00mm"
+		(property "Footprint" "TerminalBlock:TerminalBlock_Altech_AK300-2_P5.00mm"
 			(at 205.74 110.49 0)
 			(effects
